File: lit-bit/lit-bit.brd (EAGLE design)
At the start: 70 parts, among them J2 USB_MICRO_B_SMD_FEMALE, J3 ISP, U2 32U4, U3 MCP73831T, U4 ADXL345, U5 S-1335M33, U6 MCP7940N, U7 24FC1025, Y1 8MHz, Y2 32.768kHz, Y3 32.768kHz, Y4 16MHz

Commit message: working through pcb placement
Parts:
- removed C13: 100nF, SCADA_CUSTOM_LIBRARY:0603
- removed SJ1, SJ2, SJ3: (no value), microbuilder:SOLDERJUMPER_WAVE
- added JP2: sck, SparkFun-Jumpers:SMT-JUMPER_2_NO_SILK
- added JP3: mosi, SparkFun-Jumpers:SMT-JUMPER_2_NO_SILK
- added JP4: miso, SparkFun-Jumpers:SMT-JUMPER_2_NO_SILK
- added R10: 10k, SCADA_CUSTOM_LIBRARY:0603
- added SPR: LSP10, solpad:LSP10
- C10, C17, C18, C9: device SCADA_CUSTOM_LIBRARY:0805 -> SCADA_CUSTOM_LIBRARY:0603
- D1: value LED-RGSMIT -> LEDs
- U3: value MCP73831T -> 73831
- U5: value S-1335M33 -> S-1335
- moved D1 389.7 mm to (13.1, 6.99), turned to 180 degrees
- moved R2 384.5 mm to (11.8, 10.2)
- moved R1 383.9 mm to (13.3, 3.81), turned to 180 degrees
- moved C1 360.8 mm to (19.7, 14.0), turned to 180 degrees
- moved C3 355.0 mm to (22.9, 12.1), turned to 270 degrees
- moved C4 351.1 mm to (25.4, 10.2), turned to 90 degrees
- moved R5 348.3 mm to (11.8, 13.3)
- moved U3 348.0 mm to (15.7, 11.7)
- moved U2 327.8 mm to (15.2, 22.2), turned to 180 degrees
- moved R3 318.3 mm to (24.8, 14.6), turned to 180 degrees
- moved R4 311.7 mm to (23.5, 17.1), turned to 180 degrees
- moved C2 304.1 mm to (24.8, 19.7), turned to 180 degrees
- moved Y1 298.9 mm to (24.1, 23.5), turned to 90 degrees
- moved C5 287.8 mm to (0.64, 18.3), turned to 270 degrees
- moved R6 286.8 mm to (6.35, 24.8), turned to 270 degrees
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Connections:
- removed net N$10: U2.12
- removed net N$11: U2.30
- removed net N$12: U2.29
- removed net N$13: U2.28
- removed net N$14: U2.27
- removed net N$17: U2.26
- removed net N$18: U2.32
- removed net N$19: U2.25
- removed net N$8: U2.1
- net +3V3: now also JP1.3; no longer C13.1, JP1.2
- net 3V3: now also R10.2
- net ACTIVE: now also R10.1, U2.12
- net GND: now also JP1.4; no longer C13.2, JP1.1
- net MISO: now also JP4.1; no longer SJ3.1
- net MOSI: now also JP3.1; no longer SJ2.1
- net N$27: now also JP2.2; no longer SJ1.2
- net N$29: now also JP3.2; no longer SJ2.2
- net N$34: now also JP4.2; no longer SJ3.2
- net N$9: now also SPR.MP
- net NRF-RST: now also U2.26
- net RDYN: now also U2.1
- net REQN: now also U2.29
- net SCK: now also JP2.1; no longer SJ1.1
- net SCL: now also JP1.1; no longer JP1.4
- net SDA: now also JP1.2; no longer JP1.3
- net VBAT: no longer C1.1, J2.VBUS1, U3.4
- net VUSB: now also C1.1, J2.VBUS1, U3.4
Routing:
- net VBAT: track 0.00 -> 3.98 mm

Commit message: finally laid out the board
Parts:
- moved C21 68.7 mm to (2.41, 22.9), turned to 0 degrees
- moved R9 68.3 mm to (18.2, 34.9), turned to 90 degrees
- moved U$28 63.6 mm to (13.5, 39.0)
- moved C24 60.1 mm to (11.8, 40.5)
- moved C23 58.0 mm to (11.8, 38.9)
- moved C22 53.6 mm to (15.1, 38.9), turned to 0 degrees
- moved FB1 48.8 mm to (13.0, 31.1), turned to 270 degrees
- moved L3 45.5 mm to (18.4, 38.9)
- moved R10 45.2 mm to (31.2, 29.2), turned to 90 degrees
- moved L2 41.2 mm to (21.7, 38.9)
- moved C27 37.1 mm to (15.4, 35.8), turned to 0 degrees
- moved L5 35.9 mm to (15.4, 34.0)
- moved C16 35.8 mm to (26.4, 29.2), turned to 90 degrees
- moved L4 35.3 mm to (13.0, 34.9), turned to 90 degrees
- moved C15 32.8 mm to (24.0, 29.2), turned to 90 degrees
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Routing:
- net N$37: track 0.00 -> 2.13 mm
- net N$33: track 0.00 -> 1.92 mm

Commit message: acktually done with layout now, got board dimensions
Parts:
- JP1: device pinhead:1X04 -> microbuilder:1X04_ROUND
- moved J5 1.17 mm to (34.7, 13.8)
- moved J2 0.90 mm to (36.8, 10.2)
- moved C8 0.63 mm to (19.7, 12.1)
- moved D1 0.51 mm to (13.2, 8.26)
- moved C17 0.38 mm to (32.6, 40.6)
- moved Y3 0.28 mm to (32.9, 35.3)
- moved U5 0.25 mm to (28.4, 13.6)
- moved J1 0.25 mm to (19.7, 4.19)
Other:
- board outline added: 37.5 x 49.5 mm
